Commit message: Added imu, gps completely, some part of lidar

File: src/description/urdf/robot.urdf.xacro (robot description, xacro)
@@ -5,6 +5,8 @@
   <xacro:include filename="robot_control.xacro"/>
   <xacro:include filename="robot_sim.xacro"/>
+  <xacro:include filename="robot_sensors.xacro"/>
   <xacro:base/>
   <xacro:control/>
   <xacro:sim/>
+  <xacro:sensors/>
 </robot>

File: src/description/urdf/robot_base.xacro (robot description, xacro)
@@ -40,29 +40,4 @@
     <self_collide>false</self_collide>
   </gazebo>
-  <!-- ================= IMU LINK ================= -->
-<link name="imu_link"/>
-<joint name="imu_joint" type="fixed">
-  <parent link="base_link"/>
-  <child link="imu_link"/>
-  <origin xyz="0 0 0.15"/>
-</joint>
-<gazebo reference="imu_link">
-  <sensor name="imu_sensor" type="imu">
-    <always_on>true</always_on>
-    <update_rate>100</update_rate>
-    <imu>
-      <angular_velocity>
-        <x>true</x>
-        <y>true</y>
-        <z>true</z>
-      </angular_velocity>
-      <linear_acceleration>
-        <x>true</x>
-        <y>true</y>
-        <z>true</z>
-      </linear_acceleration>
-    </imu>
-  </sensor>
-</gazebo>
   <!-- ================= WHEEL MACRO ================= -->
   <xacro:macro name="wheel" params="name x y">

File: src/description/urdf/robot_sensors.xacro (robot description, xacro)
@@ -1 +1,68 @@
-<robot/>
+<?xml version="1.0"?>
+<robot xmlns:xacro="http://www.ros.org/wiki/xacro">
+  <xacro:macro name="sensors">
+    <!-- ================= IMU ================= -->
+    <gazebo reference="base_link">
+      <sensor name="imu_sensor" type="imu">
+        <always_on>true</always_on>
+        <update_rate>100</update_rate>
+        <topic>/imu</topic>
+        <imu>
+          <angular_velocity>
+            <x>true</x>
+            <y>true</y>
+            <z>true</z>
+          </angular_velocity>
+          <linear_acceleration>
+            <x>true</x>
+            <y>true</y>
+            <z>true</z>
+          </linear_acceleration>
+        </imu>
+        <plugin
+          filename="gz-sim-imu-system"
+          name="gz::sim::systems::Imu"/>
+      </sensor>
+    </gazebo>
+    <!-- ================= GPS ================= -->
+    <gazebo reference="base_link">
+      <sensor name="gps_sensor" type="navsat">
+        <always_on>true</always_on>
+        <update_rate>10</update_rate>
+        <topic>/gps</topic>
+        <plugin
+          filename="gz-sim-navsat-system"
+          name="gz::sim::systems::NavSat"/>
+      </sensor>
+    </gazebo>
+    <!-- ================= LIDAR ================= -->
+<gazebo reference="base_link">
+  <sensor name="lidar_sensor" type="gpu_lidar">
+    <always_on>true</always_on>
+    <update_rate>10</update_rate>
+    <topic>/scan</topic>
+    <gz_frame_id>base_link</gz_frame_id>
+    <lidar>
+      <scan>
+        <horizontal>
+          <samples>720</samples>
+          <resolution>1</resolution>
+          <min_angle>-3.14159</min_angle>
+          <max_angle>3.14159</max_angle>
+        </horizontal>
+      </scan>
+      <range>
+        <min>0.1</min>
+        <max>10.0</max>
+        <resolution>0.01</resolution>
+      </range>
+    </lidar>
+    <plugin
+      filename="gz-sim-sensors-system"
+      name="gz::sim::systems::Sensors">
+      <render_engine>ogre2</render_engine>
+    </plugin>
+  </sensor>
+</gazebo>
+  </xacro:macro>
+</robot>
