Commit message: more progress

File: src/description/urdf/robot_base.xacro (robot description, xacro)
@@ -92,5 +92,5 @@
       <parent link="base_link"/>
       <child link="camera_link"/>
-      <origin xyz="0.15 0 1"/>
+      <origin xyz="0.15 0 2" rpy="0 0.7 0"/>
     </joint>
     <xacro:macro name="wheel" params="name x y">

Commit message: Updated camera positioning, renamed topics, and adjusted camera orientation

File: src/description/urdf/robot_base.xacro (robot description, xacro)
@@ -181,6 +181,6 @@
       <box size="0.05 0.05 0.05"/>
     </geometry>
-    <material name="red">
-      <color rgba="1 0 0 1"/>
+    <material name="blue">
+      <color rgba="0 0 1 1"/>
     </material>
   </visual>
@@ -200,5 +200,5 @@
   <parent link="base_link"/>
   <child link="side_camera_link"/>
-  <origin xyz="0.18 0.12 0.22"/>
+  <origin xyz="0.15 0 2" rpy="0 0.4 0"/>
 </joint>
     <xacro:macro name="wheel" params="name x y">

File: src/description/urdf/robot_sensors.xacro (robot description, xacro)
@@ -41,8 +41,8 @@
     </gazebo>
     <gazebo reference="camera_link">
-      <sensor name="camera_sensor" type="camera">
+      <sensor name="turret_camera_sensor" type="camera">
         <always_on>true</always_on>
         <update_rate>30</update_rate>
-        <topic>/camera/image_raw</topic>
+        <topic>/turret_camera/image_raw</topic>
         <camera>
           <horizontal_fov>1.047</horizontal_fov>
@@ -60,8 +60,8 @@
     </gazebo>
     <gazebo reference="side_camera_link">
-  <sensor name="side_camera_sensor" type="camera">
+  <sensor name="camera_sensor" type="camera">
     <always_on>true</always_on>
     <update_rate>30</update_rate>
-    <topic>/side_camera/image_raw</topic>
+    <topic>/camera/image_raw</topic>
     <camera>
       <horizontal_fov>1.047</horizontal_fov>
